File: circuit/timer.sch (KiCad schematic (older format))
At the start: 49 parts, among them J1 Conn_01x02_Female, J2 USB_C_Receptacle_USB2.0, M1 Motor_DC, Q1 DMN3404L, SW1 SW_Push, SW2 SW_Push, U1 HDSM-541B, U2 AT32UC3L016-AUT, U3 TPS61200DRC, U4 MCP73833-AMI_UN

Commit message: v3 and coding complete
Parts:
- removed CLK1, MISO1, MOSI1, SS1: TestPoint, TestPoint:TestPoint_Pad_D4.0mm, symbol Connector:TestPoint
- removed U2: AT32UC3L016-AUT, QFP50P900X900X120-48N, symbol AT32UC3L016-AUT:AT32UC3L016-AUT
- added C7, C8: 10u, Capacitor_SMD:C_0805_2012Metric, symbol Device:C_Small
- added D4, D5: B240, Diode_SMD:D_SMB, symbol Diode:B240
- added H1, H2, H3, H4: MountingHole, MountingHole:MountingHole_4mm, symbol Mechanical:MountingHole
- added Q2: AO3401A, Package_TO_SOT_SMD:SOT-23, symbol Transistor_FET:AO3401A
- added R23: 10k, Resistor_SMD:R_0805_2012Metric, symbol Device:R_Small
- added R24: 220k, Resistor_SMD:R_0805_2012Metric, symbol Device:R_Small
- added TP3: TDI, TestPoint:TestPoint_Pad_D2.0mm, symbol Connector:TestPoint
- added TP4: TDO, TestPoint:TestPoint_Pad_D2.0mm, symbol Connector:TestPoint
- added TP5: TEST, TestPoint:TestPoint_Pad_D2.0mm, symbol Connector:TestPoint
- added U2: MSP430G2302IPW20, Package_SO:TSSOP-20_4.4x6.5mm_P0.65mm, symbol MCU_Texas_MSP430:MSP430G2302IPW20
- C4: value 22n -> 10u
- J1: LCSC (none) -> C160352
- L1: value 4.7u -> 2.2uF; footprint Inductor_SMD:L_1008_2520Metric -> Inductor_SMD:L_Wuerth_WE-PD-Typ-7345
- R10, R9: value R_Small -> 220k
- R20: value R_Small -> 10k
- SW1, SW2: LCSC (none) -> C79167
- TP1: renamed from RESET1; value TestPoint -> RESET; footprint TestPoint:TestPoint_Pad_D4.0mm -> TestPoint:TestPoint_Pad_D2.0mm
- TP6: renamed from GND1; value TestPoint -> GND; footprint TestPoint:TestPoint_Pad_D4.0mm -> TestPoint:TestPoint_Pad_D2.0mm
- TP7: renamed from 3.3; value TestPoint -> 3.3; footprint TestPoint:TestPoint_Pad_D4.0mm -> TestPoint:TestPoint_Pad_D2.0mm
- U1: footprint Display:HDSM-441B_HDSM-443B -> my-footprints:HDSM-441B_HDSM-443B-bigger
- U3: LCSC (none) -> C140320
Connections:
- net +3V3: now also C7.1, C8.2, U2.1 (DVCC)
- net +BATT: now also Q2.2 (S); no longer C1.1, C2.1, L1.2, R1.1, U3.5 (VIN), U3.6 (EN), U3.8 (PS)
- net A: now also U2.8 (P2.0)
- net B: now also U2.9 (P2.1)
- net C: now also U2.10 (P2.2)
- net CA1: now also U2.4 (TA0.1/P1.2)
- net CA2: now also U2.5 (P1.3)
- net D: now also U2.11 (P2.3)
- net DP: now also U2.18 (P2.7/XOUT)
- net E: now also U2.12 (P2.4)
- net F: now also U2.13 (P2.5)
- net G: now also U2.19 (P2.6/XIN/TA0.1)
- net GND: now also C7.2, C8.1, R23.1, R24.2, U2.20 (DVSS)
- net VDD: now also D5.2 (A), Q2.1 (G), R24.1
- net at R11.2, TP1.1: now also U2.16 (~RST~/NMI/SBWTDIO)
- net at R9.1, SW1.1: now also U2.2 (TA0CLK/ACLK/P1.0)
- net at R10.1, SW2.1: now also U2.3 (TA0.0/P1.1)
- net at Q1.1 (G), R20.1: now also U2.6 (SMCLK/TCK/TA0.2/P1.4)
- net at U3.3 (L): now also L1.2; no longer L1.1
- new net: C1.1, C2.1, D4.1 (K), D5.1 (K), L1.1, R1.1, U3.5 (VIN), U3.6 (EN), U3.8 (PS)
- new net: TP3.1, U2.14 (SDO/SCL/TDI/TCLK/TA0.1/P1.6)
- new net: TP4.1, U2.15 (SDI/SDA/TDO/TDI/P1.7)
- new net: R23.2, TP5.1, U2.17 (SBWTCK/TEST)
- new net: D4.2 (A), Q2.3 (D)
Other:
- moved on the sheet: C2, R10, R11, R9, SW1, SW2
