File: circuit/timer.kicad_pcb (KiCad board)
At the start: 2 copper layers, 60 x 60 mm, 52 parts, among them J1 Conn_01x02_Female, J2 USB_C_Receptacle_USB2.0, M1 Motor_DC, Q1 DMN3404L, SW1 SW_Push, SW2 SW_Push, U1 HDSM-541B, U2 AT32UC3L016-AUT, U3 TPS61200DRC, U4 MCP73833-AMI_UN

Commit message: v3 and coding complete
Parts:
- removed 3.3, CLK1, MISO1, MOSI1, SS1: TestPoint, TestPoint:TestPoint_Pad_D4.0mm
- removed REF** (x3): MountingHole_8.4mm_M8, MountingHole:MountingHole_8.4mm_M8
- added C7: 10u, Capacitor_SMD:C_0805_2012Metric, B.Cu at (110.8, 86.0)
- added C8: 10u, Capacitor_SMD:C_0805_2012Metric, B.Cu at (118.2, 74.8)
- added D4: B240, Diode_SMD:D_SMB, B.Cu at (102.1, 67.6)
- added D5: B240, Diode_SMD:D_SMB, B.Cu at (111.3, 92.0)
- added H1: MountingHole, MountingHole:MountingHole_4mm, F.Cu at (167.4, 71.2)
- added H2: MountingHole, MountingHole:MountingHole_4mm, F.Cu at (167.4, 80.7)
- added H3: MountingHole, MountingHole:MountingHole_4mm, F.Cu at (177.0, 71.2)
- added H4: MountingHole, MountingHole:MountingHole_4mm, F.Cu at (177.0, 80.7)
- added Q2: AO3401A, Package_TO_SOT_SMD:SOT-23, B.Cu at (106.0, 62.8)
- added R23: 10k, Resistor_SMD:R_0805_2012Metric, B.Cu at (129.6, 84.9)
- added R24: 220k, Resistor_SMD:R_0805_2012Metric, B.Cu at (110.0, 63.1)
- added TP3: TDI, TestPoint:TestPoint_Pad_D2.0mm, B.Cu at (132.8, 78.0)
- added TP4: TDO, TestPoint:TestPoint_Pad_D2.0mm, B.Cu at (136.0, 78.0)
- added TP5: TEST, TestPoint:TestPoint_Pad_D2.0mm, B.Cu at (126.3, 84.9)
- added TP7: 3.3, TestPoint:TestPoint_Pad_D2.0mm, B.Cu at (125.0, 55.0)
- C4: value 22n -> 10u
- J2: moved to B.Cu
- L1: value 4.7u -> 2.2uF; footprint Inductor_SMD:L_1008_2520Metric -> Inductor_SMD:L_Wuerth_WE-PD-Typ-7345
- R10, R9: value R_Small -> 220k
- R12, R13, R14, R15, R16, R17, R18, R19, R21, R22: value R_Small -> 75
- R20: value R_Small -> 10k
- R5: value 1k -> 5.1k
- TP1: renamed from RESET1; value TestPoint -> RESET; footprint TestPoint:TestPoint_Pad_D4.0mm -> TestPoint:TestPoint_Pad_D2.0mm
- TP6: renamed from GND1; value TestPoint -> GND; footprint TestPoint:TestPoint_Pad_D4.0mm -> TestPoint:TestPoint_Pad_D2.0mm
- U1: footprint Display:HDSM-441B_HDSM-443B -> my-footprints:HDSM-441B_HDSM-443B-bigger
- U2: value AT32UC3L016-AUT -> MSP430G2302IPW20; footprint KiCad library:QFP50P900X900X120-48N -> Package_SO:TSSOP-20_4.4x6.5mm_P0.65mm
- moved R11 18.7 mm to (137.4, 84.1), turned to 90 degrees
- moved TP1 15.9 mm to (139.2, 78.0)
- moved R3 12.1 mm to (116.5, 98.2), turned to 90 degrees
- moved D1 8.36 mm to (146.0, 80.5), turned to 0 degrees
- moved C6 8.31 mm to (120.2, 74.8), turned to 90 degrees
- moved J2 5.55 mm to (128.0, 99.0), turned to 180 degrees
- moved L1 4.95 mm to (110.8, 69.6), turned to 180 degrees
- moved J1 2.16 mm to (102.8, 74.8)
- moved C4 2.02 mm to (108.5, 86.0), turned to 270 degrees
- moved C1 1.75 mm to (114.8, 80.6)
- moved C2 1.75 mm to (114.8, 74.6)
- moved C3 1.75 mm to (107.2, 81.2)
- moved R1 1.75 mm to (114.8, 78.6)
- moved R2 1.75 mm to (114.8, 76.6)
- moved R6 1.75 mm to (111.3, 81.2)
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Connections:
- L1 pad 1: Net-(L1-Pad1) -> +BATT
- L1 pad 2: +BATT -> Net-(L1-Pad2)
- U2 pad 1: GND -> +3V3
- U2 pad 10: /G -> /C
- U2 pad 11: /A -> /D
- U2 pad 12: /F -> /E
- U2 pad 13: /C -> /F
- U2 pad 14: /B -> Net-(TP3-Pad1)
- U2 pad 15: /DP -> Net-(TP4-Pad1)
- U2 pad 16: Net-(U2-Pad16) -> Net-(R11-Pad2)
- U2 pad 17: +3V3 -> Net-(R23-Pad2)
- U2 pad 18: +3V3 -> /DP
- U2 pad 19: GND -> /G
- U2 pad 2: /CA2 -> Net-(R9-Pad1)
- U2 pad 20: Net-(U2-Pad20) -> GND
- U2 pad 3: /CA1 -> Net-(R10-Pad1)
- U2 pad 4: /D -> /CA1
- U2 pad 5: Net-(U2-Pad5) -> /CA2
- U2 pad 8: Net-(U2-Pad8) -> /A
- U2 pad 9: Net-(U2-Pad9) -> /B
- U3 pad 3: Net-(L1-Pad1) -> Net-(L1-Pad2)
Routing:
- net VDD: track 24.5 -> 90.4 mm, vias 0 -> 2
- net /F: track 58.2 -> 17.8 mm, vias 5 -> 1
- net /G: track 39.7 -> 12.0 mm, vias 3 -> 1
- net +3V3: track 185.1 -> 158.4 mm, vias 2 -> 0
- net Net-(TP4-Pad1): track 0.00 -> 17.7 mm
- net GND: track 81.1 -> 66.5 mm
- net /E: track 30.7 -> 17.5 mm
- net Net-(TP3-Pad1): track 0.00 -> 11.6 mm
- net +BATT: track 80.8 -> 92.3 mm, vias 2 -> 0
- net Net-(L1-Pad1): track 10.8 -> 0.00 mm, vias 2 -> 0
- net Net-(R11-Pad2): track 12.6 -> 23.0 mm
- net Net-(R23-Pad2): track 0.00 -> 10.4 mm
- net Net-(L1-Pad2): track 0.00 -> 10.1 mm, vias 0 -> 2
- net Net-(R10-Pad1): track 38.1 -> 46.6 mm
- net /DP: track 19.9 -> 11.7 mm, vias 3 -> 1
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Other:
- outline, holes or cut-outs redrawn
- board text added: "v3"

Commit message: ready for manufacture
Parts:
- moved H2 57.1 mm to (111.0, 90.0)
- moved H1 54.2 mm to (115.1, 57.2)
- moved H3 44.3 mm to (134.9, 57.2)
- moved H4 36.2 mm to (142.0, 90.0)
- moved D5 11.3 mm to (102.3, 85.2), turned to 180 degrees
- moved C4 6.39 mm to (114.8, 84.7), turned to 0 degrees
- moved C7 5.24 mm to (114.8, 82.6), turned to 180 degrees
- moved R22 4.07 mm to (134.4, 95.3)
- moved R11 3.31 mm to (139.2, 81.3)
- moved D2 1.99 mm to (134.2, 91.3)
- moved R3 1.78 mm to (115.9, 96.6), turned to 0 degrees
- moved D3 0.23 mm to (134.4, 95.3)
- moved R21 0.15 mm to (134.4, 93.3)
Routing:
- net Net-(D3-Pad2): track 7.31 -> 3.08 mm
- net Net-(J2-PadB5): track 9.19 -> 11.8 mm
- net +3V3: track 158.4 -> 155.9 mm
- net Net-(D2-Pad2): track 2.86 -> 4.10 mm
- net VDD: track 90.4 -> 91.6 mm, vias 2 -> 0
- net +BATT: track 92.3 -> 91.5 mm, vias 0 -> 2
- net Net-(D2-Pad1): track 10.3 -> 11.1 mm
- net GND: track 66.5 -> 66.2 mm, vias 13 -> 14
